Commit message: add use_pt_full arg and config,now we can choose use joint_traj_pt_message or joint_traj_pt_full_message to communicate with controller update readme

File: i5_a3_support/urdf/a3_macro.xacro (robot description, xacro)
@@ -204,5 +204,5 @@
 	<origin xyz="0 0 0" rpy="0 0 0"/>
 	<axis xyz="0 0 1" />
-	<limit lower="${joint1_lower_limit}" upper="${joint1_upper_limit}" effort="100" velocity="4.01425" />
+	<limit lower="${joint1_lower_limit}" upper="${joint1_upper_limit}" effort="100" velocity="1" />
 </joint>
 <joint name="${prefix}joint_2" type="revolute">
@@ -211,5 +211,5 @@
         <origin xyz="${lengthpar4} 0 ${lengthpar1}" rpy="${-PI_2} 0 0"/>
 	<axis xyz="0 0 1" />
-	<limit lower="${joint2_lower_limit}" upper="${joint2_upper_limit}" effort="100" velocity="4.01425" />
+	<limit lower="${joint2_lower_limit}" upper="${joint2_upper_limit}" effort="100" velocity="1" />
 </joint>
 <joint name="${prefix}joint_3" type="revolute">
@@ -218,5 +218,5 @@
         <origin xyz="0 ${-lengthpar2} 0" rpy="0 0 ${-PI_2}"/>
 	<axis xyz="0 0 1" />
-	<limit lower="${joint3_lower_limit}" upper="${joint3_upper_limit}" effort="100" velocity="4.36332" />
+	<limit lower="${joint3_lower_limit}" upper="${joint3_upper_limit}" effort="100" velocity="1" />
 </joint>
 <joint name="${prefix}joint_4" type="revolute">
@@ -225,5 +225,5 @@
        <origin xyz="${lengthpar3} ${lengthpar5} 0" rpy="${PI_2} 0 0"/>
 	<axis xyz="0 0 1" />
-	<limit lower="${joint4_lower_limit}" upper="${joint4_upper_limit}" effort="100" velocity="5.58505" />
+	<limit lower="${joint4_lower_limit}" upper="${joint4_upper_limit}" effort="100" velocity="1" />
 </joint>
 <joint name="${prefix}joint_5" type="revolute">
@@ -232,5 +232,5 @@
         <origin xyz="0 0 0" rpy="${PI_2} 0 0"/>
 	<axis xyz="0 0 1" />
-	<limit lower="${joint5_lower_limit}" upper="${joint5_upper_limit}" effort="5.5" velocity="5.58505" />
+	<limit lower="${joint5_lower_limit}" upper="${joint5_upper_limit}" effort="5.5" velocity="1" />
 </joint>
 <joint name="${prefix}joint_6" type="revolute">
@@ -239,5 +239,5 @@
         <origin xyz="0  ${-lengthpar6} 0" rpy="${PI_2} 0 0"/>
 	<axis xyz="0 0 1" />
-	<limit lower="${joint6_lower_limit}" upper="${joint6_upper_limit}" effort="4.6" velocity="7.3303" />
+	<limit lower="${joint6_lower_limit}" upper="${joint6_upper_limit}" effort="4.6" velocity="1" />
 </joint>
 <joint name="${prefix}joint_6-tool0" type="fixed">
